Commit message: ADD: imu accel data low pass filter

File: src/ros-ngimu/urdf/imu_urdf.urdf (robot description, URDF)
Before this commit: robot imu_urdf, 3 links, 2 joints
Links:
- removed link imu
- added link imu_link, mass 1.3729096e+00; collision box size=0.266 0.266 0.094; visual box size=0.266 0.266 0.094
Joints:
- joint base_joint: child imu -> imu_link
